Commit message: Update robot.urdf

File: urdf/robot.urdf (robot description, URDF)
Before this commit: robot my_robot, 2 links, 1 joints
Links:
- removed link link1
- added link caster_mount1; visual box size=0.03 0.02 0.01
- added link caster_mount2; visual box size=0.03 0.02 0.01
- added link caster_wheel; visual cylinder length=0.03 radius=0.01
- added link left_wheel; visual mesh filename=package://robot_description/stl/wheel.stl
- added link right_wheel; visual mesh filename=package://robot_description/stl/wheel.stl
- link base_link: mass 1 -> None; geometry visual mesh filename=package://robot_description/stl/chassis.stl
Joints:
- removed joint joint1
- added joint caster_joint1: type fixed, parent base_link, child caster_mount1, origin xyz=0.12 0.0 -0.02
- added joint caster_joint2: type fixed, parent base_link, child caster_mount2, origin xyz=-0.12 0.0 -0.02
- added joint caster_mount1_joint: type fixed, parent caster_mount1, child caster_wheel, origin xyz=0 0 0
- added joint caster_mount2_joint: type fixed, parent caster_mount2, child caster_wheel, origin xyz=0 0 0
- added joint left_wheel_joint: type continuous, parent base_link, child left_wheel, origin xyz=0.1065 0.048 0, axis 0 0 1
- added joint right_wheel_joint: type continuous, parent base_link, child right_wheel, origin xyz=-0.1065 0.048 0, axis 0 0 1
